File: KiCAD/delorean.kicad_sch (KiCad schematic)
At the start: 4 parts, among them U1 boost_conv, U2 K155ID1

Commit message: updating schematic + PCB
Parts:
- added NX2, NX3, NX4, NX5, NX6: IN-12A, footprints:IN-12, symbol IN-12:IN-12
- added R1, R2, R3, R4, R5, R6: 11kΩ, Resistor_SMD:R_0805_2012Metric_Pad1.20x1.40mm_HandSolder, symbol Device:R
- added U3, U4, U5, U6, U7: K155ID1, footprints:K155ID1, symbol K155ID1:K155ID1
Connections:
- net +5V: now reaches U1.1 (+5V)
- net +5V: now also U2.5 (VCC), U3.5 (VCC), U4.5 (VCC), U5.5 (VCC), U6.5 (VCC), U7.5 (VCC)
- net PWR: now reaches U1.2 (EN)
- net PWR: now also A1.32 (GPIO27_ADC1)
- net 170V: now reaches U1.3 (VOUT)
- net 170V: now also R1.1, R2.1, R3.1, R4.1, R5.1, R6.1
- net GND: now reaches U1.4 (GND)
- net GND: now also A1.13 (GND), A1.18 (GND), A1.23 (GND), A1.28 (GND), A1.3 (GND), A1.38 (GND), A1.8 (GND), U2.12 (GND), U3.12 (GND), U4.12 (GND), U5.12 (GND), U6.12 (GND), U7.12 (GND)
- net D1A: now reaches A1.1 (GPIO0)
- net D1A: now also U2.3 (A)
- net D2D: now reaches A1.10 (GPIO7)
- net D2D: now also U3.4 (D)
- net D3A: now reaches A1.11 (GPIO8)
- net D3A: now also U4.3 (A)
- net D3B: now reaches A1.12 (GPIO9)
- net D3B: now also U4.6 (B)
- net D3C: now reaches A1.14 (GPIO10)
- net D3C: now also U4.7 (C)
- net D3D: now reaches A1.15 (GPIO11)
- net D3D: now also U4.4 (D)
- net D4A: now reaches A1.16 (GPIO12)
- net D4A: now also U5.3 (A)
- net D4B: now reaches A1.17 (GPIO13)
- net D4B: now also U5.6 (B)
- net D4C: now reaches A1.19 (GPIO14)
- net D4C: now also U5.7 (C)
- net D1B: now reaches A1.2 (GPIO1)
- net D1B: now also U2.6 (B)
- net D4D: now reaches A1.20 (GPIO15)
- net D4D: now also U5.4 (D)
- net D5A: now reaches A1.21 (GPIO16)
- net D5A: now also U6.3 (A)
- net D5B: now reaches A1.22 (GPIO17)
- net D5B: now also U6.6 (B)
- net D5C: now reaches A1.24 (GPIO18)
- net D5C: now also U6.7 (C)
- net D5D: now reaches A1.25 (GPIO19)
- net D5D: now also U6.4 (D)
- net D6A: now reaches A1.26 (GPIO20)
- net D6A: now also U7.3 (A)
- net D6B: now reaches A1.27 (GPIO21)
- net D6B: now also U7.6 (B)
- net D6C: now reaches A1.29 (GPIO22)
- net D6C: now also U7.7 (C)
- net D6D: now reaches A1.31 (GPIO26_ADC0)
- net D6D: now also U7.4 (D)
- net D1C: now reaches A1.4 (GPIO2)
- net D1C: now also U2.7 (C)
- net D1D: now reaches A1.5 (GPIO3)
- net D1D: now also U2.4 (D)
- net D2A: now reaches A1.6 (GPIO4)
- net D2A: now also U3.3 (A)
- net D2B: now reaches A1.7 (GPIO5)
- net D2B: now also U3.6 (B)
- net D2C: now reaches A1.9 (GPIO6)
- net D2C: now also U3.7 (C)
- net at NX1.1 (A): now also R1.2
- net at NX1.10 (2): now also U2.8 (2)
- net at NX1.11 (1): now also U2.15 (1)
- net at NX1.2 (0): now also U2.16 (0)
- net at NX1.3 (9): now also U2.2 (9)
- net at NX1.4 (8): now also U2.1 (8)
- net at NX1.5 (7): now also U2.10 (7)
- net at NX1.6: now also U2.11 (6)
- net at NX1.7 (5): now also U2.14 (5)
- net at NX1.8 (4): now also U2.13 (4)
- net at NX1.9 (3): now also U2.9 (3)
- new net: NX2.4 (8), U3.1 (8)
- new net: NX2.5 (7), U3.10 (7)
- new net: NX2.6, U3.11 (6)
- new net: NX2.8 (4), U3.13 (4)
- new net: NX2.7 (5), U3.14 (5)
- new net: NX2.11 (1), U3.15 (1)
- new net: NX2.2 (0), U3.16 (0)
- new net: NX2.3 (9), U3.2 (9)
- new net: NX2.10 (2), U3.8 (2)
- new net: NX2.9 (3), U3.9 (3)
- new net: NX6.1 (A), R6.2
- new net: NX6.10 (2), U7.8 (2)
- new net: NX6.11 (1), U7.15 (1)
- new net: NX6.2 (0), U7.16 (0)
- new net: NX6.3 (9), U7.2 (9)
- new net: NX6.4 (8), U7.1 (8)
- new net: NX6.5 (7), U7.10 (7)
- new net: NX6.6, U7.11 (6)
- new net: NX6.7 (5), U7.14 (5)
- new net: NX6.8 (4), U7.13 (4)
- new net: NX6.9 (3), U7.9 (3)
- new net: NX5.4 (8), U6.1 (8)
- new net: NX5.5 (7), U6.10 (7)
- new net: NX5.6, U6.11 (6)
- new net: NX5.8 (4), U6.13 (4)
- new net: NX5.7 (5), U6.14 (5)
- new net: NX5.11 (1), U6.15 (1)
- new net: NX5.2 (0), U6.16 (0)
- new net: NX5.3 (9), U6.2 (9)
- new net: NX5.10 (2), U6.8 (2)
- new net: NX5.9 (3), U6.9 (3)
- new net: NX5.1 (A), R5.2
- new net: NX4.1 (A), R4.2
- new net: NX4.10 (2), U5.8 (2)
- new net: NX4.11 (1), U5.15 (1)
- new net: NX4.2 (0), U5.16 (0)
- new net: NX4.3 (9), U5.2 (9)
- new net: NX4.4 (8), U5.1 (8)
- new net: NX4.5 (7), U5.10 (7)
- new net: NX4.6, U5.11 (6)
- new net: NX4.7 (5), U5.14 (5)
- new net: NX4.8 (4), U5.13 (4)
- new net: NX4.9 (3), U5.9 (3)
- new net: NX3.4 (8), U4.1 (8)
- new net: NX3.5 (7), U4.10 (7)
- new net: NX3.6, U4.11 (6)
- new net: NX3.8 (4), U4.13 (4)
- new net: NX3.7 (5), U4.14 (5)
- new net: NX3.11 (1), U4.15 (1)
- new net: NX3.2 (0), U4.16 (0)
- new net: NX3.3 (9), U4.2 (9)
- new net: NX3.10 (2), U4.8 (2)
- new net: NX3.9 (3), U4.9 (3)
- new net: NX3.1 (A), R3.2
- new net: NX2.1 (A), R2.2
Other:
- note added: "digit 1"
- note added: "digit 2"
- note added: "digit 3"
- note added: "digit 4"
- note added: "digit 5"
- note added: "digit 6"
- company: (none) -> Hack Club
- title: (none) -> The DeLorean
- moved on the sheet: A1, NX1, U1

Commit message: routed PCB
Parts:
- A1: footprint Module:RaspberryPi_Pico_W_SMD_HandSolder -> Module:RaspberryPi_Pico_Common_THT
Changed lines of the file:
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@@
 			)
 		)
-		(property "Footprint" "Module:RaspberryPi_Pico_W_SMD_HandSolder"
+		(property "Footprint" "Module:RaspberryPi_Pico_Common_THT"
 			(at 51.435 196.215 0)
 			(effects
