File: KiCAD/delorean.kicad_pcb (KiCad board)
At the start: 2 copper layers, 4 parts, among them U1 boost_conv, U2 K155ID1

Commit message: updating schematic + PCB
Parts:
- added NX2: IN-12A, footprints:IN-12, F.Cu at (134.6, 67.0)
- added NX3: IN-12A, footprints:IN-12, F.Cu at (164.0, 67.0)
- added NX4: IN-12A, footprints:IN-12, F.Cu at (185.5, 67.0)
- added NX5: IN-12A, footprints:IN-12, F.Cu at (215.0, 67.0)
- added NX6: IN-12A, footprints:IN-12, F.Cu at (236.5, 67.0)
- added R1: 11kΩ, Resistor_SMD:R_0805_2012Metric_Pad1.20x1.40mm_HandSolder, F.Cu at (99.0, 59.0)
- added R2: 11kΩ, Resistor_SMD:R_0805_2012Metric_Pad1.20x1.40mm_HandSolder, F.Cu at (149.0, 59.0)
- added R3: 11kΩ, Resistor_SMD:R_0805_2012Metric_Pad1.20x1.40mm_HandSolder, F.Cu at (149.5, 71.0)
- added R4: 11kΩ, Resistor_SMD:R_0805_2012Metric_Pad1.20x1.40mm_HandSolder, F.Cu at (199.5, 59.5)
- added R5: 11kΩ, Resistor_SMD:R_0805_2012Metric_Pad1.20x1.40mm_HandSolder, F.Cu at (200.0, 72.0)
- added R6: 11kΩ, Resistor_SMD:R_0805_2012Metric_Pad1.20x1.40mm_HandSolder, F.Cu at (251.5, 73.0)
- added U3: K155ID1, footprints:K155ID1, F.Cu at (137.3, 92.5)
- added U4: K155ID1, footprints:K155ID1, F.Cu at (163.7, 92.8)
- added U5: K155ID1, footprints:K155ID1, F.Cu at (187.7, 93.4)
- added U6: K155ID1, footprints:K155ID1, F.Cu at (214.7, 93.3)
- added U7: K155ID1, footprints:K155ID1, F.Cu at (241.1, 93.6)
- A1: moved to B.Cu
- moved A1 167.2 mm to (227.9, 111.2), turned to 90 degrees
- moved NX1 20.0 mm to (113.1, 67.0)
- moved U2 17.4 mm to (112.8, 91.7), turned to 180 degrees
- moved U1 15.1 mm to (122.6, 117.6), turned to 180 degrees
Connections:
- A1 pad 1: unconnected-(A1-GPIO0-Pad1) -> D1A
- A1 pad 10: unconnected-(A1-GPIO7-Pad10) -> D2D
- A1 pad 11: unconnected-(A1-GPIO8-Pad11) -> D3A
- A1 pad 12: unconnected-(A1-GPIO9-Pad12) -> D3B
- A1 pad 13: Net-(A1-GND-Pad13) -> GND
- A1 pad 14: unconnected-(A1-GPIO10-Pad14) -> D3C
- A1 pad 15: unconnected-(A1-GPIO11-Pad15) -> D3D
- A1 pad 16: unconnected-(A1-GPIO12-Pad16) -> D4A
- A1 pad 17: unconnected-(A1-GPIO13-Pad17) -> D4B
- A1 pad 18: Net-(A1-GND-Pad13) -> GND
- A1 pad 19: unconnected-(A1-GPIO14-Pad19) -> D4C
- A1 pad 2: unconnected-(A1-GPIO1-Pad2) -> D1B
- A1 pad 20: unconnected-(A1-GPIO15-Pad20) -> D4D
- A1 pad 21: unconnected-(A1-GPIO16-Pad21) -> D5A
- A1 pad 22: unconnected-(A1-GPIO17-Pad22) -> D5B
- A1 pad 23: Net-(A1-GND-Pad13) -> GND
- A1 pad 24: unconnected-(A1-GPIO18-Pad24) -> D5C
- A1 pad 25: unconnected-(A1-GPIO19-Pad25) -> D5D
- A1 pad 26: unconnected-(A1-GPIO20-Pad26) -> D6A
- A1 pad 27: unconnected-(A1-GPIO21-Pad27) -> D6B
- A1 pad 28: Net-(A1-GND-Pad13) -> GND
- A1 pad 29: unconnected-(A1-GPIO22-Pad29) -> D6C
- A1 pad 3: Net-(A1-GND-Pad13) -> GND
- A1 pad 31: unconnected-(A1-GPIO26_ADC0-Pad31) -> D6D
- A1 pad 32: unconnected-(A1-GPIO27_ADC1-Pad32) -> PWR
- A1 pad 38: Net-(A1-GND-Pad13) -> GND
- A1 pad 4: unconnected-(A1-GPIO2-Pad4) -> D1C
- A1 pad 5: unconnected-(A1-GPIO3-Pad5) -> D1D
- A1 pad 6: unconnected-(A1-GPIO4-Pad6) -> D2A
- A1 pad 7: unconnected-(A1-GPIO5-Pad7) -> D2B
- A1 pad 8: Net-(A1-GND-Pad13) -> GND
- A1 pad 9: unconnected-(A1-GPIO6-Pad9) -> D2C
- NX1 pad 1: unconnected-(NX1-A-Pad1) -> Net-(NX1-A)
- NX1 pad 10: unconnected-(NX1-2-Pad10) -> Net-(NX1-2)
- NX1 pad 11: unconnected-(NX1-1-Pad11) -> Net-(NX1-1)
- NX1 pad 2: unconnected-(NX1-0-Pad2) -> Net-(NX1-0)
- NX1 pad 3: unconnected-(NX1-9-Pad3) -> Net-(NX1-9)
- NX1 pad 4: unconnected-(NX1-8-Pad4) -> Net-(NX1-8)
- NX1 pad 5: unconnected-(NX1-7-Pad5) -> Net-(NX1-7)
- NX1 pad 6: unconnected-(NX1-Pad6) -> Net-(U2-6)
- NX1 pad 7: unconnected-(NX1-5-Pad7) -> Net-(NX1-5)
- NX1 pad 8: unconnected-(NX1-4-Pad8) -> Net-(NX1-4)
- NX1 pad 9: unconnected-(NX1-3-Pad9) -> Net-(NX1-3)
- U1 pad 1: unconnected-(U1-+5V-Pad1) -> +5V
- U1 pad 2: unconnected-(U1-EN-Pad2) -> PWR
- U1 pad 3: unconnected-(U1-VOUT-Pad3) -> 170V
- U1 pad 4: unconnected-(U1-GND-Pad4) -> GND
- U2 pad 1: unconnected-(U2-8-Pad1) -> Net-(NX1-8)
- U2 pad 10: unconnected-(U2-1-Pad10) -> Net-(NX1-7)
- U2 pad 11: unconnected-(U2-5-Pad11) -> Net-(U2-6)
- U2 pad 12: unconnected-(U2-4-Pad12) -> GND
- U2 pad 13: unconnected-(U2-GND-Pad13) -> Net-(NX1-4)
- U2 pad 14: unconnected-(U2-6-Pad14) -> Net-(NX1-5)
- U2 pad 15: unconnected-(U2-7-Pad15) -> Net-(NX1-1)
- U2 pad 16: unconnected-(U2-3-Pad16) -> Net-(NX1-0)
- U2 pad 2: unconnected-(U2-9-Pad2) -> Net-(NX1-9)
- U2 pad 3: unconnected-(U2-A-Pad3) -> D1A
- U2 pad 4: unconnected-(U2-D-Pad4) -> D1D
- U2 pad 5: unconnected-(U2-VCC-Pad5) -> +5V
- U2 pad 6: unconnected-(U2-B-Pad6) -> D1B
- U2 pad 7: unconnected-(U2-C-Pad7) -> D1C
- U2 pad 8: unconnected-(U2-2-Pad8) -> Net-(NX1-2)
- U2 pad 9: unconnected-(U2-0-Pad9) -> Net-(NX1-3)
Other:
- board outline added: 159.7 x 76.8 mm

Commit message: routed PCB
Parts:
- A1: value RaspberryPi_Pico_W -> Raspberry Pi Pico W; footprint Module:RaspberryPi_Pico_W_SMD_HandSolder -> Module:RaspberryPi_Pico_Common_THT; moved to F.Cu
- moved R5 31.6 mm to (224.6, 52.1)
- moved R3 30.9 mm to (173.9, 52.1)
- moved A1 25.6 mm to (252.1, 102.9), turned to -90 degrees
- moved R6 21.4 mm to (246.9, 52.0)
- moved U1 18.5 mm to (104.3, 120.2), turned to 90 degrees
- moved R4 7.29 mm to (199.5, 52.2)
- moved R2 6.82 mm to (149.0, 52.2)
- moved R1 6.78 mm to (99.5, 52.2)
- moved U2 3.24 mm to (109.7, 92.5), turned to 0 degrees
- moved U4 2.02 mm to (161.7, 92.5)
- moved U7 1.22 mm to (240.7, 92.5)
- moved U3 1.16 mm to (136.2, 92.5)
- moved U5 0.91 mm to (187.7, 92.5)
- moved U6 0.83 mm to (214.9, 92.5)
Routing:
- net GND: track 0.00 -> 255.7 mm
- net 170V: track 0.00 -> 217.5 mm
- net +5V: track 0.00 -> 174.0 mm
- net D1A: track 0.00 -> 152.9 mm
- net D1D: track 0.00 -> 142.5 mm, vias 0 -> 1
- net D1B: track 0.00 -> 142.3 mm
- net D1C: track 0.00 -> 133.2 mm
- net PWR: track 0.00 -> 121.2 mm
- net D2A: track 0.00 -> 116.1 mm, vias 0 -> 1
- net D2B: track 0.00 -> 105.6 mm, vias 0 -> 1
- net D2C: track 0.00 -> 105.3 mm, vias 0 -> 2
- net D2D: track 0.00 -> 99.4 mm, vias 0 -> 1
- net D3A: track 0.00 -> 73.8 mm, vias 0 -> 2
- net D3B: track 0.00 -> 65.1 mm, vias 0 -> 1
- net D3D: track 0.00 -> 64.8 mm, vias 0 -> 2
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- added copper zone on B.Cu, net GND
- added copper zone on F.Cu, net GND
Other:
- board size 159.7 x 76.8 mm -> 160.3 x 77.5 mm
- board text added: "R5"

Commit message: silkscreen
Parts:
- added G***: LOGO, LOGO, F.Cu at (131.5, 112.5)
Other:
- board text added: "meghana inc."

Commit message: PCB update + imgs
Parts:
- A1: value Raspberry Pi Pico W -> RaspberryPi_Pico_W
Routing:
- net D2C: track 105.3 -> 100.2 mm
Changed lines of the file:
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@@
 			)
 		)
+		(model "${KIPRJMOD}/libs/steps/IN-12 Nixie Tube.stp"
+			(offset
+				(xyz 0 0 -8.5)
+			)
+			(scale
+				(xyz 1 1 1)
+			)
+			(rotate
+				(xyz -0 -0 -0)
+			)
+		)
 	)
 	(footprint "footprints:K155ID1"
@@
 			)
 		)
+		(model "${KIPRJMOD}/libs/steps/IN-12 Nixie Tube.stp"
+			(offset
+				(xyz 0 0 -8.5)
+			)
+			(scale
+				(xyz 1 1 1)
+			)
+			(rotate
+				(xyz -0 -0 -0)
+			)
+		)
 	)
 	(footprint "footprints:K155ID1"
@@
 			)
 		)
-		(property "Value" "Raspberry Pi Pico W"
+		(property "Value" "RaspberryPi_Pico_W"
 			(at 8.89 52.07 270)
 			(unlocked yes)
@@
 		)
 		(property "Datasheet" "https://datasheets.raspberrypi.com/picow/pico-w-datasheet.pdf"
-			(at 8.89 24.13 270)
+			(at 8.89 24.13 90)
 			(layer "F.Fab")
 			(hide yes)
@@
 		)
 		(property "Description" "Versatile and inexpensive wireless microcontroller module powered by RP2040 dual-core Arm Cortex-M0+ processor up to 133 MHz, 264kB SRAM, 2MB QSPI flash, Infineon CYW43439 2.4GHz 802.11n wireless LAN; also supports Raspberry Pi Pico 2 W"
-			(at 8.89 24.13 270)
+			(at 8.89 24.13 90)
 			(layer "F.Fab")
 			(hide yes)
@@
 			)
 		)
+		(model "${KIPRJMOD}/libs/steps/RaspberryPi Pico W v2.step"
+			(offset
+				(xyz 9 1.5 -0.5)
+			)
+			(scale
+				(xyz 1 1 1)
+			)
+			(rotate
+				(xyz -0 -0 -0)
+			)
+		)
 	)
 	(footprint "LOGO"
@@
 		(model "${KIPRJMOD}/libs/steps/IN-12 Nixie Tube.STEP"
 			(offset
-				(xyz 0 0 0)
+				(xyz 0 0 -8.5)
 			)
 			(scale
@@
 			)
 			(rotate
-				(xyz 0 0 0)
+				(xyz -0 -0 -0)
+			)
+		)
+		(model "${KIPRJMOD}/libs/steps/IN-12 Nixie Tube.stp"
+			(offset
+				(xyz 0 0 -8.5)
+			)
+			(scale
+				(xyz 1 1 1)
+			)
+			(rotate
+				(xyz -0 -0 -0)
 			)
 		)
@@
 			)
 		)
+		(model "${KIPRJMOD}/libs/steps/IN-12 Nixie Tube.stp"
+			(offset
+				(xyz 0 0 -8.5)
+			)
+			(scale
+				(xyz 1 1 1)
+			)
+			(rotate
+				(xyz -0 -0 -0)
+			)
+		)
 	)
 	(footprint "footprints:IN-12"
@@
 			)
 		)
+		(model "${KIPRJMOD}/libs/steps/IN-12 Nixie Tube.stp"
+			(offset
+				(xyz 0 0 -8.5)
+			)
+			(scale
+				(xyz 1 1 1)
+			)
+			(rotate
+				(xyz -0 -0 -0)
+			)
+		)
 	)
 	(footprint "footprints:IN-12"
@@
 			)
 		)
+		(model "${KIPRJMOD}/libs/steps/IN-12 Nixie Tube.stp"
+			(offset
+				(xyz 0 -0.5 -8.5)
+			)
+			(scale
+				(xyz 1 1 1)
+			)
+			(rotate
+				(xyz -0 -0 -0)
+			)
+		)
 	)
 	(footprint "Resistor_SMD:R_0805_2012Metric_Pad1.20x1.40mm_HandSolder"
@@
 		(net 11)
 	)
-	(segment
-		(start 145.3268 92.5322)
-		(end 144.4108 93.4482)
-		(width 0.2)
-		(layer "F.Cu")
-		(net 11)
-	)
-	(segment
-		(start 144.4108 93.4482)
-		(end 145.3268 92.5322)
-		(width 0.2)
-		(layer "F.Cu")
-		(net 11)
-	)
 	(via
 		(at 227.5084 91.9884)
@@
 		(width 0.2)
 		(layer "B.Cu")
-		(net 11)
-	)
-	(segment
-		(start 144.4108 93.4482)
-		(end 145.3268 92.5322)
-		(width 0.2)
-		(layer "B.Cu")
-		(net 11)
-	)
-	(segment
-		(start 145.3268 92.5322)
-		(end 144.4108 93.4482)
-		(width 0.2)
-		(layer "B.Cu")

Commit message: pcb update + img
Parts:
- removed the G*** at (131.5, 112.5)
- added G***: LOGO, LOGO, F.Cu at (127.4, 113.2)
- added G***: LOGO, LOGO, F.Cu at (145.2, 113.8)
Other:
- board text added: "DELOREAN"
- board text added: "meghana inc. // highway 2025"
- board text added: "the"

Commit message: render stuff
Parts:
- moved G*** 2.09 mm to (143.2, 114.4)
